File: HW2/hmwk2/hmwk2.sch (EAGLE design)
At the start: 22 parts, among them J1 USB_MINI-B_SMT

Commit message: updated board
Parts:
- removed J1: USB_MINI-B_SMT, components:USB_MINI-B_SMT
- added K1: 651005136521, components:651005136521
Connections:
- net D+: now also K1.D+; no longer J1.D+
- net D-: now also K1.D-; no longer J1.D-
- net GND: now also K1.GND; no longer J1.GND, J1.SHIELD
- net ID: now also K1.ID; no longer J1.ID
- net VIN: now also K1.VCC; no longer J1.VBUS
Changed lines of the file:
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@@
 <parts>
 <part name="IC1" library="components" deviceset="DIL28" device="-3"/>
-<part name="J1" library="components" deviceset="USB_MINI-B" device="_SMT"/>
 <part name="R1" library="components" deviceset="R-US_" device="0207/10" value="10kohm"/>
 <part name="C1" library="components" deviceset="C-US" device="025-025X050" value="0.1uf"/>
@@
 <part name="C6" library="components" deviceset="C-US" device="025-025X050" value="0.1uf"/>
 <part name="GND14" library="components" deviceset="GND" device=""/>
-<part name="GND15" library="components" deviceset="GND" device=""/>
 <part name="R3" library="components" deviceset="R-US_" device="0207/10" value="10kohm"/>
 <part name="+3V3" library="components" deviceset="+3V3" device=""/>
@@
 <part name="J3" library="components" deviceset="CONN_08" device="&quot;"/>
 <part name="J4" library="components" deviceset="CONN_08" device="&quot;"/>
+<part name="K1" library="components" deviceset="651005136521" device=""/>
 </parts>
 <sheets>
@@
 <instances>
 <instance part="IC1" gate="G$1" x="45.72" y="43.18"/>
-<instance part="J1" gate="G$1" x="-15.24" y="78.74" rot="R180"/>
 <instance part="R1" gate="G$1" x="27.94" y="58.42"/>
 <instance part="C1" gate="G$1" x="17.78" y="66.04" rot="R90"/>
@@
 <instance part="C6" gate="G$1" x="68.58" y="45.72" rot="R90"/>
 <instance part="GND14" gate="1" x="76.2" y="45.72" rot="R90"/>
-<instance part="GND15" gate="1" x="-27.94" y="78.74" rot="R270"/>
 <instance part="R3" gate="G$1" x="20.32" y="-5.08" rot="R270"/>
 <instance part="+3V3" gate="G$1" x="20.32" y="2.54"/>
@@
 <instance part="J3" gate="G$1" x="38.1" y="-2.54"/>
 <instance part="J4" gate="G$1" x="66.04" y="-2.54"/>
+<instance part="K1" gate="G$1" x="-53.34" y="78.74" rot="R180"/>
 </instances>
 <busses>
@@
 </segment>
 <segment>
-<pinref part="J1" gate="G$1" pin="D-"/>
-<wire x1="-10.16" y1="76.2" x2="-5.08" y2="76.2" width="0.1524" layer="91"/>
-<label x="-2.54" y="76.2" size="1.778" layer="95"/>
+<pinref part="K1" gate="G$1" pin="D-"/>
+<wire x1="-45.72" y1="76.2" x2="-40.64" y2="76.2" width="0.1524" layer="91"/>
+<label x="-43.18" y="76.2" size="1.778" layer="95"/>
 </segment>
 </net>
@@
 </segment>
 <segment>
-<pinref part="J1" gate="G$1" pin="D+"/>
-<wire x1="-10.16" y1="78.74" x2="-5.08" y2="78.74" width="0.1524" layer="91"/>
-<label x="-5.08" y="78.74" size="1.778" layer="95"/>
+<pinref part="K1" gate="G$1" pin="D+"/>
+<wire x1="-45.72" y1="78.74" x2="-40.64" y2="78.74" width="0.1524" layer="91"/>
+<label x="-43.18" y="78.74" size="1.778" layer="95"/>
 </segment>
 </net>
@@
 </segment>
 <segment>
-<pinref part="J1" gate="G$1" pin="ID"/>
-<wire x1="-10.16" y1="81.28" x2="-5.08" y2="81.28" width="0.1524" layer="91"/>
-<label x="-5.08" y="81.28" size="1.778" layer="95"/>
+<pinref part="K1" gate="G$1" pin="ID"/>
+<wire x1="-45.72" y1="81.28" x2="-40.64" y2="81.28" width="0.1524" layer="91"/>
+<label x="-43.18" y="81.28" size="1.778" layer="95"/>
 </segment>
 </net>
 <net name="GND" class="0">
-<segment>
-<pinref part="J1" gate="G$1" pin="GND"/>
-<wire x1="-10.16" y1="83.82" x2="-5.08" y2="83.82" width="0.1524" layer="91"/>
-<label x="-5.08" y="83.82" size="1.778" layer="95"/>
-</segment>
 <segment>
 <pinref part="GND2" gate="1" pin="GND"/>
@@
 </segment>
 <segment>
-<pinref part="J1" gate="G$1" pin="SHIELD"/>
-<wire x1="-22.86" y1="78.74" x2="-25.4" y2="78.74" width="0.1524" layer="91"/>
-<pinref part="GND15" gate="1" pin="GND"/>
-</segment>
-<segment>
 <pinref part="S1" gate="BEF1" pin="O"/>
 <wire x1="-81.28" y1="25.4" x2="-81.28" y2="27.94" width="0.1524" layer="91"/>
@@
 <pinref part="R4" gate="G$1" pin="1"/>
 <wire x1="35.56" y1="76.2" x2="40.64" y2="76.2" width="0.1524" layer="91"/>
+</segment>
+<segment>
+<pinref part="K1" gate="G$1" pin="GND"/>
+<wire x1="-45.72" y1="83.82" x2="-40.64" y2="83.82" width="0.1524" layer="91"/>
+<label x="-43.18" y="83.82" size="1.778" layer="95"/>
 </segment>
 </net>
@@
 <net name="VIN" class="0">
 <segment>
-<pinref part="J1" gate="G$1" pin="VBUS"/>
-<label x="-7.62" y="71.12" size="1.778" layer="95"/>
-<wire x1="-10.16" y1="73.66" x2="-5.08" y2="73.66" width="0.1524" layer="91"/>
-</segment>
-<segment>
 <pinref part="S1" gate="BEF1" pin="S"/>
 <wire x1="-76.2" y1="25.4" x2="-76.2" y2="27.94" width="0.1524" layer="91"/>
@@
 <label x="73.66" y="-7.62" size="1.778" layer="95"/>
 </segment>
-</net>
+<segment>
+<pinref part="K1" gate="G$1" pin="VCC"/>
+<wire x1="-45.72" y1="73.66" x2="-40.64" y2="73.66" width="0.1524" layer="91"/>
+<label x="-43.18" y="73.66" size="1.778" layer="95"/>
+</segment>
+</net>
